File: e1/src/Test_sur_uno/simulation_avec_arduino_uno.brd (EAGLE design)
At the start: 68.6 x 53.3 mm, 8 parts

Commit message: mise a jour du test
Parts:
- removed Rpot2: 250k‎Ω, AUTODESK_CIRCUITS_BREADBOARD:B25V
- moved BAT1 12.7 mm to (5.00, 86.3)
- moved R3 12.7 mm to (5.00, 60.9)
- moved S1 12.7 mm to (5.00, 73.6)
- moved R1 12.7 mm to (5.00, 48.2)
- moved R2 12.7 mm to (5.00, 35.5)
